Commit message: Add files via upload

File: my_robot_description/urdf/02-description.xacro (robot description, xacro)
@@ -3,13 +3,10 @@
     <xacro:property name="body_length" value="1.0" />
     <xacro:property name="body_width" value="0.55" />
-    <xacro:property name="body_height" value="0.25" />
+    <xacro:property name="body_height" value="0.1" />
     <xacro:property name="body_mass" value="10" />
-    <xacro:property name="wheel_width" value="0.15" />
-    <xacro:property name="wheel_radius" value="0.15" />
+    <xacro:property name="wheel_width" value="0.1" />
+    <xacro:property name="wheel_radius" value="0.1" />
     <xacro:property name="wheel_mass" value="1" />
     <!---->
-    <xacro:macro name="set_bl_as_parent_link">
-        <parent link="base_link" />
-    </xacro:macro>
     <!--DEFINITION DE MACRO DES ROUE-->
     <xacro:macro name="create_wheel" params="position">
